Commit message: Add missing STL's. Updeate sensor.xacro

File: urdf/fixposition_holder.xacro (robot description, xacro)
@@ -2,5 +2,5 @@
 <robot xmlns:xacro="http://www.ros.org/wiki/xacro">
   <!-- Define a macro for the bridge joint -->
-  <xacro:macro name="bridge_joint" params="xyz rpy">
+  <xacro:macro name="fixposition_holder" params="parent xyz rpy">
     <link name="Fixposion_base">
       <inertial>
@@ -12,5 +12,5 @@
         <origin xyz="0 0 0" rpy="0 0 0"/>
         <geometry>
-          <mesh filename="$(find j8_xacro_model)/meshes/Fixposion_base.STL"/>
+          <mesh filename="$(find fixposition_sensor_pkg)/meshes/Fixposion_base.STL"/>
         </geometry>
         <material name=""><color rgba="0.25098 0.25098 0.25098 0.2"/></material>
@@ -19,5 +19,5 @@
         <origin xyz="0 0 0" rpy="0 0 0"/>
         <geometry>
-          <mesh filename="$(find j8_xacro_model)/meshes/Fixposion_base.STL"/>
+          <mesh filename="$(find fixposition_sensor_pkg)/meshes/Fixposion_base.STL"/>
         </geometry>
       </collision>
@@ -26,5 +26,5 @@
     <joint name="Bridge_fixposion_base_joint" type="fixed">
       <origin xyz="${xyz}" rpy="${rpy}"/>
-      <parent link="Bridge"/>
+      <parent link="${parent}"/>
       <child link="Fixposion_base"/>
       <axis xyz="0 0 0"/>
@@ -40,5 +40,5 @@
         <origin xyz="0 0 0" rpy="0 0 0"/>
         <geometry>
-          <mesh filename="$(find j8_xacro_model)/meshes/Left_fixposition_feet.STL"/>
+          <mesh filename="$(find fixposition_sensor_pkg)/meshes/Left_fixposition_feet.STL"/>
         </geometry>
         <material name=""><color rgba="0.64706 0.92549 0.90196 1"/></material>
@@ -47,5 +47,5 @@
         <origin xyz="0 0 0" rpy="0 0 0"/>
         <geometry>
-          <mesh filename="$(find j8_xacro_model)/meshes/Left_fixposition_feet.STL"/>
+          <mesh filename="$(find fixposition_sensor_pkg)/meshes/Left_fixposition_feet.STL"/>
         </geometry>
       </collision>
@@ -68,5 +68,5 @@
         <origin xyz="0 0 0" rpy="0 0 0"/>
         <geometry>
-          <mesh filename="$(find j8_xacro_model)/meshes/Left_fixposition_holder.STL"/>
+          <mesh filename="$(find fixposition_sensor_pkg)/meshes/Left_fixposition_holder.STL"/>
         </geometry>
         <material name=""><color rgba="0.79216 0.81961 0.93333 1"/></material>
@@ -75,5 +75,5 @@
         <origin xyz="0 0 0" rpy="0 0 0"/>
         <geometry>
-          <mesh filename="$(find j8_xacro_model)/meshes/Left_fixposition_holder.STL"/>
+          <mesh filename="$(find fixposition_sensor_pkg)/meshes/Left_fixposition_holder.STL"/>
         </geometry>
       </collision>
@@ -96,5 +96,5 @@
         <origin xyz="0 0 0" rpy="0 0 0"/>
         <geometry>
-          <mesh filename="$(find j8_xacro_model)/meshes/Central_fixposition_feet.STL"/>
+          <mesh filename="$(find fixposition_sensor_pkg)/meshes/Central_fixposition_feet.STL"/>
         </geometry>
         <material name=""><color rgba="0.64706 0.92549 0.90196 1"/></material>
@@ -103,5 +103,5 @@
         <origin xyz="0 0 0" rpy="0 0 0"/>
         <geometry>
-          <mesh filename="$(find j8_xacro_model)/meshes/Central_fixposition_feet.STL"/>
+          <mesh filename="$(find fixposition_sensor_pkg)/meshes/Central_fixposition_feet.STL"/>
         </geometry>
       </collision>
@@ -124,5 +124,5 @@
         <origin xyz="0 0 0" rpy="0 0 0"/>
         <geometry>
-          <mesh filename="$(find j8_xacro_model)/meshes/Central_fixposition_holder.STL"/>
+          <mesh filename="$(find fixposition_sensor_pkg)/meshes/Central_fixposition_holder.STL"/>
         </geometry>
         <material name=""><color rgba="0.79216 0.81961 0.93333 1"/></material>
@@ -131,5 +131,5 @@
         <origin xyz="0 0 0" rpy="0 0 0"/>
         <geometry>
-          <mesh filename="$(find j8_xacro_model)/meshes/Central_fixposition_holder.STL"/>
+          <mesh filename="$(find fixposition_sensor_pkg)/meshes/Central_fixposition_holder.STL"/>
         </geometry>
       </collision>
@@ -152,5 +152,5 @@
         <origin xyz="0 0 0" rpy="0 0 0"/>
         <geometry>
-          <mesh filename="$(find j8_xacro_model)/meshes/Right_fixposition_feet.STL"/>
+          <mesh filename="$(find fixposition_sensor_pkg)/meshes/Right_fixposition_feet.STL"/>
         </geometry>
         <material name=""><color rgba="0.64706 0.92549 0.90196 1"/></material>
@@ -159,5 +159,5 @@
         <origin xyz="0 0 0" rpy="0 0 0"/>
         <geometry>
-          <mesh filename="$(find j8_xacro_model)/meshes/Right_fixposition_feet.STL"/>
+          <mesh filename="$(find fixposition_sensor_pkg)/meshes/Right_fixposition_feet.STL"/>
         </geometry>
       </collision>
@@ -180,5 +180,5 @@
         <origin xyz="0 0 0" rpy="0 0 0"/>
         <geometry>
-          <mesh filename="$(find j8_xacro_model)/meshes/Right_fixposition_holder.STL"/>
+          <mesh filename="$(find fixposition_sensor_pkg)/meshes/Right_fixposition_holder.STL"/>
         </geometry>
         <material name=""><color rgba="0.79216 0.81961 0.93333 1"/></material>
@@ -187,5 +187,5 @@
         <origin xyz="0 0 0" rpy="0 0 0"/>
         <geometry>
-          <mesh filename="$(find j8_xacro_model)/meshes/Right_fixposition_holder.STL"/>
+          <mesh filename="$(find fixposition_sensor_pkg)/meshes/Right_fixposition_holder.STL"/>
         </geometry>
       </collision>

File: urdf/fixposition_main.xacro (robot description, xacro)
@@ -2,9 +2,9 @@
 <robot xmlns:xacro="http://www.ros.org/wiki/xacro" name="fixposition_sensor">
   <!-- Include individual components -->
-  <xacro:include filename="$(find fixposition)/urdf/fixposition_holder.xacro"/>
-  <xacro:include filename="$(find fixposition)/urdf/fixposition_sensor.xacro"/>
+  <xacro:include filename="$(find fixposition_sensor_pkg)/urdf/fixposition_holder.xacro"/>
+  <xacro:include filename="$(find fixposition_sensor_pkg)/urdf/fixposition_sensor.xacro"/>
   <!-- Macro to instantiate the full sensor setup -->
   <xacro:macro name="fixposition_full_setup" params="parent xyz rpy">
-    <xacro:fixposition_holder parent="${parent}" xyz="${xyz}" rpy="${rpy}"/>
+     <xacro:fixposition_holder parent="${parent}" xyz="${xyz}" rpy="${rpy}"/>
     <xacro:fixposition_sensor frame_joint_xyz="0 0.035 0.0526" frame_joint_rpy="-1.5708 0 3.1416"/>
   </xacro:macro>

File: urdf/fixposition_sensor.xacro (robot description, xacro)
@@ -2,5 +2,5 @@
 <robot xmlns:xacro="http://www.ros.org/wiki/xacro" name="fixposition_sensor">
   <xacro:macro name="fixposition_sensor" params="frame_joint_xyz frame_joint_rpy">
-    <!-- Fix_position_metal_frame link -->
+    <!-- Link for the Fix_position_metal_frame -->
     <link name="Fix_position_metal_frame">
       <inertial>
@@ -25,5 +25,6 @@
       </collision>
     </link>
-    <xacro:set_gazebo_color link_name="Fix_position_metal_frame" r="0.5" g="0.5" b="0.5"/> <!-- Grey-->
+    <xacro:set_gazebo_color link_name="Fix_position_metal_frame" r="0.5" g="0.5" b="0.5"/> <!-- Set color for Fix_position_metal_frame in Gazebo -->
+    <!-- Joint for the Fix_position_metal_frame -->
     <joint name="Fix_position_metal_frame_joint" type="fixed">
       <origin xyz="${frame_joint_xyz}" rpy="${frame_joint_rpy}" />
@@ -32,4 +33,5 @@
       <axis xyz="0 0 0" />
     </joint>
+    <!-- Link and Joint for the Fix_position_left_antenna -->
     <link name="Fix_position_left_antenna">
       <inertial>
@@ -54,113 +56,65 @@
       </collision>
     </link>
-    <xacro:set_gazebo_color link_name="Fix_position_left_antenna" r="0.0" g="0.0" b="0.0"/> <!-- Black-->
-  <joint
-    name="Fix_position_metal_frame_left_antenna_joint"
-    type="fixed">
-    <origin
-      xyz="-0.146 -0.033263 0"
-      rpy="-1.5708 0 3.1416" />
-    <parent
-      link="Fix_position_metal_frame" />
-    <child
-      link="Fix_position_left_antenna" />
-    <axis
-      xyz="0 0 0" />
-  </joint>
-  <link
-    name="Fixposition_right_antenna">
-    <inertial>
-      <origin
-        xyz="-0.015 0.026394 2.2204E-16"
-        rpy="0 0 0" />
-      <mass
-        value="0.034976" />
-      <inertia
-        ixx="1.0676E-05"
-        ixy="2.2713E-20"
-        ixz="-9.1301E-22"
-        iyy="3.5788E-06"
-        iyz="6.8941E-22"
-        izz="1.0676E-05" />
-    </inertial>
-    <visual>
-      <origin
-        xyz="0 0 0"
-        rpy="0 0 0" />
-      <geometry>
-        <mesh
-          filename="$(find j8_xacro_model)/meshes/Fixposition_right_antenna.STL" />
-      </geometry>
-      <material
-        name="">
-        <color
-          rgba="0.054902 0.054902 0.054902 1" />
-      </material>
-    </visual>
-    <collision>
-      <origin
-        xyz="0 0 0"
-        rpy="0 0 0" />
-      <geometry>
-        <mesh
-          filename="$(find j8_xacro_model)/meshes/Fixposition_right_antenna.STL" />
-      </geometry>
-    </collision>
-  </link>
-  <xacro:set_gazebo_color link_name="Fixposition_right_antenna" r="0.0" g="0.0" b="0.0"/> <!-- Black-->
-  <joint
-    name="Fix_position_metal_frame_right_antenna_joint"
-    type="fixed">
-    <origin
-      xyz="0.174 -0.033263 0"
-      rpy="-1.5708 0 3.1416" />
-    <parent
-      link="Fix_position_metal_frame" />
-    <child
-      link="Fixposition_right_antenna" />
-    <axis
-      xyz="0 0 0" />
-  </joint>
-  <link
-    name="Fixposition_lower_case">
-    <inertial>
-      <origin
-        xyz="-0.014 0.001488 -0.0029226"
-        rpy="0 0 0" />
-      <mass
-        value="0.036156" />
-      <inertia
-        ixx="4.5219E-05"
-        ixy="-1.032E-19"
-        ixz="1.071E-19"
-        iyy="7.4014E-05"
-        iyz="-3.7348E-09"
-        izz="2.8848E-05" />
-    </inertial>
-    <visual>
-      <origin
-        xyz="0 0 0"
-        rpy="0 0 0" />
-      <geometry>
-        <mesh
-          filename="$(find j8_xacro_model)/meshes/Fixposition_lower_case.STL" />
-      </geometry>
-      <material
-        name="">
-        <color
-          rgba="0.62745 0.62745 0.62745 1" />
-      </material>
-    </visual>
-    <collision>
-      <origin
-        xyz="0 0 0"
-        rpy="0 0 0" />
-      <geometry>
-        <mesh
-          filename="$(find j8_xacro_model)/meshes/Fixposition_lower_case.STL" />
-      </geometry>
-    </collision>
-  </link>
-    <xacro:set_gazebo_color link_name="Fixposition_lower_case" r="0.5" g="0.5" b="0.5"/> <!-- Grey-->
+    <xacro:set_gazebo_color link_name="Fix_position_left_antenna" r="0.0" g="0.0" b="0.0"/> <!-- Set color for Fix_position_left_antenna in Gazebo -->
+    <joint name="Fix_position_metal_frame_left_antenna_joint" type="fixed">
+      <origin xyz="-0.146 -0.033263 0" rpy="-1.5708 0 3.1416" />
+      <parent link="Fix_position_metal_frame" />
+      <child link="Fix_position_left_antenna" />
+      <axis xyz="0 0 0" />
+    </joint>
+    <!-- Link and Joint for the Fixposition_right_antenna -->
+    <link name="Fixposition_right_antenna">
+      <inertial>
+        <origin xyz="-0.015 0.026394 2.2204E-16" rpy="0 0 0" />
+        <mass value="0.034976" />
+        <inertia ixx="1.0676E-05" ixy="2.2713E-20" ixz="-9.1301E-22" iyy="3.5788E-06" iyz="6.8941E-22" izz="1.0676E-05" />
+      </inertial>
+      <visual>
+        <origin xyz="0 0 0" rpy="0 0 0" />
+        <geometry>
+          <mesh filename="$(find j8_xacro_model)/meshes/Fixposition_right_antenna.STL" />
+        </geometry>
+        <material name="">
+          <color rgba="0.054902 0.054902 0.054902 1" />
+        </material>
+      </visual>
+      <collision>
+        <origin xyz="0 0 0" rpy="0 0 0" />
+        <geometry>
+          <mesh filename="$(find j8_xacro_model)/meshes/Fixposition_right_antenna.STL" />
+        </geometry>
+      </collision>
+    </link>
+    <xacro:set_gazebo_color link_name="Fixposition_right_antenna" r="0.0" g="0.0" b="0.0"/> <!-- Set color for Fixposition_right_antenna in Gazebo -->
+    <joint name="Fix_position_metal_frame_right_antenna_joint" type="fixed">
+      <origin xyz="0.174 -0.033263 0" rpy="-1.5708 0 3.1416" />
+      <parent link="Fix_position_metal_frame" />
+      <child link="Fixposition_right_antenna" />
+      <axis xyz="0 0 0" />
+    </joint>
+    <!-- Link and Joint for the Fixposition_lower_case -->
+    <link name="Fixposition_lower_case">
+      <inertial>
+        <origin xyz="-0.014 0.001488 -0.0029226" rpy="0 0 0" />
+        <mass value="0.036156" />
+        <inertia ixx="4.5219E-05" ixy="-1.032E-19" ixz="1.071E-19" iyy="7.4014E-05" iyz="-3.7348E-09" izz="2.8848E-05" />
+      </inertial>
+      <visual>
+        <origin xyz="0 0 0" rpy="0 0 0" />
+        <geometry>
+          <mesh filename="$(find j8_xacro_model)/meshes/Fixposition_lower_case.STL" />
+        </geometry>
+        <material name="">
+          <color rgba="0.62745 0.62745 0.62745 1" />
+        </material>
+      </visual>
+      <collision>
+        <origin xyz="0 0 0" rpy="0 0 0" />
+        <geometry>
+          <mesh filename="$(find j8_xacro_model)/meshes/Fixposition_lower_case.STL" />
+        </geometry>
+      </collision>
+    </link>
+    <xacro:set_gazebo_color link_name="Fixposition_lower_case" r="0.5" g="0.5" b="0.5"/> <!-- Set color for Fixposition_lower_case in Gazebo -->
     <joint name="Fixposition_lower_case_joint" type="fixed">
       <origin xyz="0 0 0" rpy="-1.5708 0 3.1416" />
@@ -169,51 +123,151 @@
       <axis xyz="0 0 0" />
     </joint>
+    <!-- Link and Joint for the Fixposition_upper_case -->
+    <link name="Fixposition_upper_case">
+      <inertial>
+        <origin xyz="-0.012785 0.011907 -0.0047657" rpy="0 0 0" />
+        <mass value="0.080046" />
+        <inertia ixx="0.00014944" ixy="1.4031E-07" ixz="1.8093E-06" iyy="0.00024178" iyz="-6.1595E-08" izz="0.00010365" />
+      </inertial>
+      <visual>
+        <origin xyz="0 0 0" rpy="0 0 0" />
+        <geometry>
+          <mesh filename="$(find j8_xacro_model)/meshes/Fixposition_upper_case.STL" />
+        </geometry>
+        <material name="">
+          <color rgba="0.89412 0.91373 0.92941 1" />
+        </material>
+      </visual>
+      <collision>
+        <origin xyz="0 0 0" rpy="0 0 0" />
+        <geometry>
+          <mesh filename="$(find j8_xacro_model)/meshes/Fixposition_upper_case.STL" />
+        </geometry>
+      </collision>
+    </link>
+    <xacro:set_gazebo_color link_name="Fixposition_upper_case" r="0.5" g="0.5" b="0.5"/> <!-- Set color for Fixposition_upper_case in Gazebo -->
+    <joint name="Fixposition_upper_case_joint" type="fixed">
+      <origin xyz="0 0 -0.01" rpy="-1.5708 0 3.1416" />
+      <parent link="Fix_position_metal_frame" />
+      <child link="Fixposition_upper_case" />
+      <axis xyz="0 0 0" />
+    </joint>
+    <!-- Link and Joint for the Fixposition_camera -->
+    <link name="Fixposition_camera">
+      <inertial>
+        <origin xyz="-0.014 3.3307E-16 0.00050429" rpy="0 0 0" />
+        <mass value="0.00054956" />
+        <inertia ixx="1.2517E-08" ixy="-1.5542E-22" ixz="-1.5936E-22" iyy="4.8525E-08" iyz="-2.4248E-25" izz="6.0952E-08" />
+      </inertial>
+      <visual>
+        <origin xyz="0 0 0" rpy="0 0 0" />
+        <geometry>
+          <mesh filename="$(find j8_xacro_model)/meshes/Fixposition_camera.STL" />
+        </geometry>
+        <material name="">
+          <color rgba="0 0 0 1" />
+        </material>
+      </visual>
+      <collision>
+        <origin xyz="0 0 0" rpy="0 0 0" />
+        <geometry>
+          <mesh filename="$(find j8_xacro_model)/meshes/Fixposition_camera.STL" />
+        </geometry>
+      </collision>
+    </link>
+    <xacro:set_gazebo_color link_name="Fixposition_camera" r="0.0" g="0.0" b="0.0"/> <!-- Set color for Fixposition_camera in Gazebo -->
+    <joint name="Fixposition_camera_joint" type="fixed">
+      <origin xyz="0 0.006 0.061" rpy="0 0 0" />
+      <parent link="Fixposition_upper_case" />
+      <child link="Fixposition_camera" />
+      <axis xyz="0 0 0" />
+    </joint>
+    <!-- Sensor configuration for the right antenna -->
     <gazebo reference="Fixposition_right_antenna">
       <sensor name="Fixposition_right_antenna" type="gps">
         <always_on>true</always_on>
-        <update_rate>8.0</update_rate>
+        <update_rate>5.0</update_rate>
         <plugin name="fix_right_gps_node" filename="libgazebo_ros_gps_sensor.so">
-         <remapping>~/out:=/fixposition/gnss1</remapping>
+          <remapping>~/out:=/fixposition/gnss1</remapping>
           <remapping>~/vel:=/fixposition/gnss1/vel</remapping>
-          <frame_name>Fixposition_right_antenna</frame_name>
-        </plugin>
-      </sensor>
-  </gazebo>
+          <frame_name>GNSS1</frame_name>
+        </plugin>
+      </sensor>
+    </gazebo>
+    <!-- Sensor configuration for the left antenna -->
     <gazebo reference="Fix_position_left_antenna">
       <sensor name="Fix_position_left_antenna" type="gps">
         <always_on>true</always_on>
-        <update_rate>8.0</update_rate>
+        <update_rate>5.0</update_rate>
         <plugin name="fix_left_gps_node" filename="libgazebo_ros_gps_sensor.so">
-         <remapping>~/out:=/fixposition/gnss2</remapping>
+          <remapping>~/out:=/fixposition/gnss2</remapping>
           <remapping>~/vel:=/fixposition/gnss2/vel</remapping>
-          <frame_name>Fix_position_left_antenna</frame_name>
-        </plugin>
-      </sensor>
-    </gazebo>
-<gazebo reference="Fixposition_upper_case">
-    <sensor name="fixposition_imu" type="imu">
+          <frame_name>GNSS2</frame_name>
+        </plugin>
+      </sensor>
+    </gazebo>
+    <!-- IMU sensor configuration for the upper case -->
+    <gazebo reference="Fixposition_upper_case">
+      <sensor name="fixposition_imu" type="imu">
+        <always_on>true</always_on>
+        <update_rate>45</update_rate>
+        <plugin name="fixposition_imu_node" filename="libgazebo_ros_imu_sensor.so">
+          <ros>
+            <namespace>/fixposition</namespace>
+            <remapping>~/out:=corrimu</remapping>
+            <frame_name>FP_VRTK</frame_name>
+          </ros>
+          <initial_orientation_as_reference>false</initial_orientation_as_reference>
+        </plugin>
+      </sensor>
+    </gazebo>
+    <!-- Sensor configuration for POI GPS -->
+    <gazebo reference="base_link">
+      <sensor name="FP_poi_gps" type="gps">
+        <always_on>true</always_on>
+        <update_rate>4.0</update_rate>
+        <plugin name="fix_poi_node" filename="libgazebo_ros_gps_sensor.so">
+          <remapping>~/out:=/fixposition/navsatfix</remapping>
+          <remapping>~/vel:=/fixposition/navsatfix/vel</remapping>
+          <frame_name>FP_POI</frame_name>
+        </plugin>
+      </sensor>
+    </gazebo>
+    <!-- GPS sensor configuration for the lower case -->
+    <gazebo>
+        <plugin name="fixposition_tf_node" filename="libgazebo_ros_fixposition_pugin.so">
+            <update_frequency>200.0</update_frequency>
+        </plugin>
+    </gazebo>
+  </xacro:macro>
+    <!-- IMU sensor configuration for the upper case -->
+    <gazebo reference="base_link">
+      <sensor name="fixposition_poi_imu" type="imu">
         <always_on>true</always_on>
         <update_rate>200</update_rate>
-        <plugin name="fixposition_imu_node" filename="libgazebo_ros_imu_sensor.so">
-            <ros>
-                <namespace>/fixposition</namespace>
-                <remapping>~/out:=corrimu</remapping>
-            </ros>
-            <initial_orientation_as_reference>false</initial_orientation_as_reference>
-        </plugin>
-    </sensor>
-</gazebo>
-<gazebo reference="Fixposition_lower_case">
-    <sensor name="fixposition_tf" type="gps">
+        <plugin name="fixposition_raw_imu_node" filename="libgazebo_ros_imu_sensor.so">
+          <ros>
+            <namespace>/fixposition</namespace>
+            <remapping>~/out:=raw_imu</remapping>
+            <frame_name>FP_VRTK</frame_name>
+          </ros>
+          <initial_orientation_as_reference>false</initial_orientation_as_reference>
+        </plugin>
+      </sensor>
+    </gazebo>
+        <!-- IMU sensor configuration for the upper case -->
+    <gazebo reference="base_link">
+      <sensor name="fixposition_raw_imu" type="imu">
         <always_on>true</always_on>
         <update_rate>200</update_rate>
-        <plugin name="fixposition_tf_node" filename="libgazebo_ros_fixposition_plugin.so">
-                    <ros>
-                <namespace>/test</namespace>
-                <remapping>~/out:=corrimu</remapping>
-            </ros>
-        </plugin>
-    </sensor>
-</gazebo>
-  </xacro:macro>
+        <plugin name="fixposition_poi_imu_node" filename="libgazebo_ros_imu_sensor.so">
+          <ros>
+            <namespace>/fixposition</namespace>
+            <remapping>~/out:=poiimu</remapping>
+            <frame_name>FP_POI</frame_name>
+          </ros>
+          <initial_orientation_as_reference>false</initial_orientation_as_reference>
+        </plugin>
+      </sensor>
+    </gazebo>
 </robot>
